Commit message: add kuka

File: Model/Model_URDF_SLDASM/KUKA/urdf/KUKA.urdf (robot description, URDF)
Before this commit: robot KUKA, 7 links, 6 joints
Links:
- link Link1: geometry collision mesh filename=package://kuka/meshes/Link1.STL; visual mesh filename=package://kuka/meshes/Link1.STL
- link Link2: geometry collision mesh filename=package://kuka/meshes/Link2.STL; visual mesh filename=package://kuka/meshes/Link2.STL
- link Link3: geometry collision mesh filename=package://kuka/meshes/Link3.STL; visual mesh filename=package://kuka/meshes/Link3.STL
- link Link4: geometry collision mesh filename=package://kuka/meshes/Link4.STL; visual mesh filename=package://kuka/meshes/Link4.STL
- link Link5: geometry collision mesh filename=package://kuka/meshes/Link5.STL; visual mesh filename=package://kuka/meshes/Link5.STL
- link Link6: geometry collision mesh filename=package://kuka/meshes/Link6.STL; visual mesh filename=package://kuka/meshes/Link6.STL
- link base_link: geometry collision mesh filename=package://kuka/meshes/base_link.STL; visual mesh filename=package://kuka/meshes/base_link.STL
