Commit message: update kuka

File: ws_moveit_dt/src/kuka/urdf/kuka.urdf (robot description, URDF)
Before this commit: robot kuka, 7 links, 6 joints
Links:
- link Link5: mass 0.442067197041385 -> 0.442067197041382
Joints:
- joint Joint1: axis 0 0 0 -> 0 0 -1
- joint Joint2: axis 0 0 0 -> 0 1 0
- joint Joint3: axis 0 0 0 -> 0 1 0
- joint Joint4: axis 0 0 0 -> -1 0 0
- joint Joint5: axis 0 0 0 -> 0 -1 0
- joint Joint6: axis 0 0 0 -> -1 0 0
