Commit message: update kuka

File: Model/Model_URDF_SLDASM/kuka/urdf/kuka.urdf (robot description, URDF)
Before this commit: robot kuka, 7 links, 6 joints
Links:
- link Link1: mass 6.2752643308886 -> 6.27526433045034
- link Link2: mass 7.36258357526296 -> 7.36258419634408
- link Link3: mass 2.90698496201672 -> 2.90698496298682
- link Link4: mass 2.75654211573202 -> 2.75654211573085
- link Link5: mass 0.442067197041368 -> 0.442067197041385
- link Link6: mass 0.0139949492210213 -> 0.0139949492210216
Joints:
- joint Joint1: axis 0 0 -1 -> 0 0 0; origin xyz=0.8275 -1.3595 -0.29335 rpy=1.5708 0 0 -> xyz=0.99274 -1.1143 1.2159 rpy=0 0 0
- joint Joint2: axis 0 1 0 -> 0 0 0; origin xyz=0.025 0 0.183 rpy=0 0 0 -> xyz=0.025 0 0.4 rpy=0 0 0
- joint Joint3: axis 0 1 0 -> 0 0 0; origin xyz=0 0 0.315 rpy=0 0 0 -> xyz=0 0.003 0.315 rpy=0 0 0
- joint Joint4: axis -1 0 0 -> 0 0 0; origin xyz=0.10695 0.003 0.035 rpy=0 0 0 -> xyz=-0.025 0 0.035 rpy=0 0 0
- joint Joint5: axis 0 -1 0 -> 0 0 0; origin xyz=0.25805 0 0 rpy=0 0 0 -> xyz=0.39 0 0 rpy=0 0 0
- joint Joint6: axis -1 0 0 -> 0 0 0; origin xyz=0.0665 0 0 rpy=0 0 0 -> xyz=-0.39 0 0 rpy=0 0 0

Commit message: update kuka

File: Model/Model_URDF_SLDASM/kuka/urdf/kuka.urdf (robot description, URDF)
Before this commit: robot kuka, 7 links, 6 joints
Links:
- link Link1: mass 6.27526433045034 -> 6.27526433045052
- link Link2: mass 7.36258419634408 -> 7.36258419830385
- link Link3: mass 2.90698496298682 -> 2.90698496734874
- link Link4: mass 2.75654211573085 -> 2.75654210425904
- link Link5: mass 0.442067197041382 -> 0.442067197041371
- link Link6: mass 0.0139949492210216 -> 0.0139949492210214
Joints:
- joint Joint1: axis 0 0 -1 -> 0 0 1; origin xyz=0.99274 -1.1143 1.2159 rpy=0 0 0 -> xyz=0.8275 -0.43219 1.3595 rpy=0 0 0
- joint Joint2: axis 0 1 0 -> 0 -1 0; origin xyz=0.025 0 0.4 rpy=0 0 0 -> xyz=0.025 0 0.183 rpy=0 0 0
- joint Joint3: axis 0 1 0 -> 0 -1 0; origin xyz=0 0.003 0.315 rpy=0 0 0 -> xyz=0 0 0.315 rpy=0 0 0
- joint Joint4: origin xyz=-0.025 0 0.035 rpy=0 0 0 -> xyz=0.10695 0.003 0.035 rpy=0 0 0
- joint Joint5: axis 0 -1 0 -> 0 1 0; origin xyz=0.39 0 0 rpy=0 0 0 -> xyz=0.25805 0 0 rpy=0 0 0
- joint Joint6: axis -1 0 0 -> 1 0 0; origin xyz=-0.39 0 0 rpy=0 0 0 -> xyz=0.0665 0 0 rpy=0 0 0
