Commit message: update kuka_urdf

File: Model/Model_URDF_SLDASM/kuka_urdf/urdf/kuka_urdf.urdf (robot description, URDF)
Before this commit: robot kuka_urdf, 7 links, 6 joints
Links:
- link Link1: mass 6.27526433045052 -> 6.2753
- link Link2: mass 7.36258419830385 -> 7.3626
- link base_link: mass 171.3125135409 -> 171.31
Joints:
- joint Joint1: limit lower=0 upper=0 effort=0 velocity=0 -> lower=0 upper=0 effort=500 velocity=1
- joint Joint2: limit lower=0 upper=0 effort=0 velocity=0 -> lower=0 upper=0 effort=500 velocity=1
- joint Joint3: limit lower=0 upper=0 effort=0 velocity=0 -> lower=0 upper=0 effort=500 velocity=1
- joint Joint4: limit lower=0 upper=0 effort=0 velocity=0 -> lower=0 upper=0 effort=500 velocity=1
- joint Joint5: limit lower=0 upper=0 effort=0 velocity=0 -> lower=0 upper=0 effort=500 velocity=1
- joint Joint6: limit lower=0 upper=0 effort=0 velocity=0 -> lower=0 upper=0 effort=500 velocity=1

Commit message: add ws_kuka_v2

File: Model/Model_URDF_SLDASM/kuka_urdf/urdf/kuka_urdf.urdf (robot description, URDF)
Before this commit: robot kuka_urdf, 7 links, 6 joints
Links:
- added link Link7, mass 0.0139949492210214; collision mesh filename=package://kuka_urdf/meshes/Link7.STL; visual mesh filename=package://kuka_urdf/meshes/Link7.STL
- link Link1: mass 6.2753 -> 13.310335827662
- link Link2: mass 7.3626 -> 6.27526433045033
- link Link3: mass 2.90698496734874 -> 7.36258419830387
- link Link4: mass 2.75654210425904 -> 2.90698496202437
- link Link5: mass 0.442067197041372 -> 2.75654211573216
- link Link6: mass 0.0139949492210214 -> 0.442067197041368
- link base_link: mass 171.31 -> 156.699273713239
Joints:
- added joint Joint7: type revolute, parent Link6, child Link7, origin xyz=0.0665 0 0 rpy=0 0 0, axis 1 0 0, limit lower=-6.28 upper=6.28 effort=500 velocity=2
- joint Joint1: axis 0 0 1 -> 0 0 0; limit lower=0 upper=0 effort=500 velocity=1 -> lower=-2 upper=2 effort=0 velocity=1; origin xyz=0.8275 -0.43219 1.3595 rpy=0 0 0 -> xyz=0.8275 -0.43219 1.1355 rpy=3.1416 0 1.5708; type revolute -> continuous
- joint Joint2: axis 0 -1 0 -> 0 0 1; limit lower=0 upper=0 effort=500 velocity=1 -> lower=-6.28 upper=6.28 effort=500 velocity=2; origin xyz=0.025 0 0.183 rpy=0 0 0 -> xyz=0 0 -0.224 rpy=3.1416 0 1.5708
- joint Joint3: limit lower=0 upper=0 effort=500 velocity=1 -> lower=-6.28 upper=6.28 effort=500 velocity=2; origin xyz=0 0 0.315 rpy=0 0 0 -> xyz=0.025 0 0.183 rpy=0 0 0
- joint Joint4: axis -1 0 0 -> 0 -1 0; limit lower=0 upper=0 effort=500 velocity=1 -> lower=-6.28 upper=6.28 effort=500 velocity=2; origin xyz=0.10695 0.003 0.035 rpy=0 0 0 -> xyz=0 0 0.315 rpy=0 0 0
- joint Joint5: axis 0 1 0 -> -1 0 0; limit lower=0 upper=0 effort=500 velocity=1 -> lower=-6.28 upper=6.28 effort=500 velocity=2; origin xyz=0.25805 0 0 rpy=0 0 0 -> xyz=0.10695 0.003 0.035 rpy=0 0 0
- joint Joint6: axis 1 0 0 -> 0 1 0; limit lower=0 upper=0 effort=500 velocity=1 -> lower=-6.28 upper=6.28 effort=500 velocity=2; origin xyz=0.0665 0 0 rpy=0 0 0 -> xyz=0.25805 0 0 rpy=0 0 0

File: ws_kuka_v2/src/kuka_urdf/urdf/kuka_urdf.urdf (robot description, URDF)
Before this commit: robot kuka_urdf, 8 links, 7 joints
Links:
- link Link2: mass 6.27526433045052 -> 6.27526433045033
- link Link3: mass 7.36258419830385 -> 7.36258419830387
- link Link4: mass 2.90698496734874 -> 2.90698496202437
- link Link5: mass 2.75654210425904 -> 2.75654211573216
- link Link6: mass 0.442067197041371 -> 0.442067197041368
Joints:
- joint Joint1: axis 0 1 0 -> 0 0 0; limit lower=-100 upper=100 effort=500 velocity=2 -> lower=-2 upper=2 effort=0 velocity=1; origin xyz=0.8275 -0.43219 1.3595 rpy=0 0 0 -> xyz=0.8275 -0.43219 1.1355 rpy=3.1416 0 1.5708
- joint Joint2: origin xyz=0.025 0 0.183 rpy=0 0 0 -> xyz=0 0 -0.224 rpy=3.1416 0 1.5708
- joint Joint3: origin xyz=0 0 0.315 rpy=0 0 0 -> xyz=0.025 0 0.183 rpy=0 0 0
- joint Joint4: origin xyz=0.10695 0.003 0.035 rpy=0 0 0 -> xyz=0 0 0.315 rpy=0 0 0
- joint Joint5: origin xyz=0.25805 0 0 rpy=0 0 0 -> xyz=0.10695 0.003 0.035 rpy=0 0 0
- joint Joint6: origin xyz=0.0665 0 0 rpy=0 0 0 -> xyz=0.25805 0 0 rpy=0 0 0
- joint Joint7: origin xyz=0 0 0 rpy=0 0 0 -> xyz=0.0665 0 0 rpy=0 0 0

Commit message: modify ws_kuka_v2

File: Model/Model_URDF_SLDASM/kuka_urdf/urdf/kuka_urdf.urdf (robot description, URDF)
Before this commit: robot kuka_urdf, 8 links, 7 joints
Links:
- removed link Link7
- link Link6: mass 0.442067197041368 -> 0.45606214626239
Joints:
- removed joint Joint7
- joint Joint1: axis 0 0 0 -> 1 0 0; limit lower=-2 upper=2 effort=0 velocity=1 -> lower=-2 upper=2 effort=500 velocity=1; type continuous -> prismatic
