Commit message: modify ws_kuka_v1_1

File: ws_kuka_v1_1/src/kuka_urdf/urdf/kuka_urdf.urdf (robot description, URDF)
Before this commit: robot kuka_urdf, 7 links, 6 joints
Links:
- link Link1: mass 6.27526433045051 -> 6.27526433045052
- link Link5: mass 0.442067197041372 -> 0.442067197041371
- link base_link: mass 171.312513540901 -> 170.009626249841

Commit message: modify ws_kuka_v1_1

File: ws_kuka_v1_1/src/kuka_urdf/urdf/kuka_urdf.urdf (robot description, URDF)
Before this commit: robot kuka_urdf, 7 links, 6 joints
Links:
- removed link Link1
- removed link Link2
- removed link Link3
- removed link Link4
- removed link Link5
- removed link Link6
- added link link1, mass 6.27526433045052; collision mesh filename=package://kuka_urdf/meshes/link1.STL; visual mesh filename=package://kuka_urdf/meshes/link1.STL
- added link link2, mass 7.36258419830385; collision mesh filename=package://kuka_urdf/meshes/link2.STL; visual mesh filename=package://kuka_urdf/meshes/link2.STL
- added link link3, mass 2.90698496734874; collision mesh filename=package://kuka_urdf/meshes/link3.STL; visual mesh filename=package://kuka_urdf/meshes/link3.STL
- added link link4, mass 2.75654210425904; collision mesh filename=package://kuka_urdf/meshes/link4.STL; visual mesh filename=package://kuka_urdf/meshes/link4.STL
- added link link5, mass 0.442067197041371; collision mesh filename=package://kuka_urdf/meshes/link5.STL; visual mesh filename=package://kuka_urdf/meshes/link5.STL
- added link link6, mass 0.0139949492210214; collision mesh filename=package://kuka_urdf/meshes/link6.STL; visual mesh filename=package://kuka_urdf/meshes/link6.STL
- link base_link: mass 170.009626249841 -> 170.00957643814
Joints:
- removed joint Joint1
- removed joint Joint2
- removed joint Joint3
- removed joint Joint4
- removed joint Joint5
- removed joint Joint6
- added joint joint1: type revolute, parent base_link, child link1, origin xyz=0.8275 -0.43219 1.3595 rpy=0 0 0, axis 0 0 1, limit lower=-6.28 upper=6.28 effort=500 velocity=2
- added joint joint2: type revolute, parent link1, child link2, origin xyz=0.025 0 0.183 rpy=0 0 0, axis 0 -1 0, limit lower=-6.28 upper=6.28 effort=500 velocity=2
- added joint joint3: type revolute, parent link2, child link3, origin xyz=0 0 0.315 rpy=0 0 0, axis 0 -1 0, limit lower=-6.28 upper=6.28 effort=500 velocity=2
- added joint joint4: type revolute, parent link3, child link4, origin xyz=0.10695 0.003 0.035 rpy=0 0 0, axis -1 0 0, limit lower=-6.28 upper=6.28 effort=500 velocity=2
- added joint joint5: type revolute, parent link4, child link5, origin xyz=0.25805 0 0 rpy=0 0 0, axis 0 1 0, limit lower=-6.28 upper=6.28 effort=500 velocity=2
- added joint joint6: type revolute, parent link5, child link6, origin xyz=0.0665 0 0 rpy=0 0 0, axis 1 0 0, limit lower=-6.28 upper=6.28 effort=500 velocity=2

Commit message: modify ws_kuka_v1_1

File: ws_kuka_v1_1/src/kuka_urdf/urdf/kuka_urdf.urdf (robot description, URDF)
Before this commit: robot kuka_urdf, 7 links, 6 joints
Links:
- link base_link: mass 170.00957643814 -> 170.0096095409
- link link5: mass 0.442067197041371 -> 0.442067197041372

Commit message: update ws_kuka_v1_1

File: ws_kuka_v1_1/src/kuka_urdf/urdf/kuka_urdf.urdf (robot description, URDF)
Before this commit: robot kuka_urdf, 7 links, 6 joints
Links:
- link base_link: mass 170.0096095409 -> 170.00957643814
- link link5: mass 0.442067197041372 -> 0.442067197041371
Joints:
- joint joint1: limit lower=-6.28 upper=6.28 effort=500 velocity=2 -> lower=-12.56 upper=12.56 effort=500 velocity=2
- joint joint2: limit lower=-6.28 upper=6.28 effort=500 velocity=2 -> lower=-12.56 upper=12.56 effort=500 velocity=2
- joint joint3: limit lower=-6.28 upper=6.28 effort=500 velocity=2 -> lower=-12.56 upper=12.56 effort=500 velocity=2
- joint joint4: limit lower=-6.28 upper=6.28 effort=500 velocity=2 -> lower=-12.56 upper=12.56 effort=500 velocity=2
- joint joint5: limit lower=-6.28 upper=6.28 effort=500 velocity=2 -> lower=-12.56 upper=12.56 effort=500 velocity=2
- joint joint6: limit lower=-6.28 upper=6.28 effort=500 velocity=2 -> lower=-12.56 upper=12.56 effort=500 velocity=2
