Commit message: modify kuka_urdf.urdf

File: ws_kuka/src/kuka_urdf/urdf/kuka_urdf.urdf (robot description, URDF)
Before this commit: robot kuka_urdf, 8 links, 7 joints
Joints:
- joint Joint1: limit lower=-3.14 upper=3.14 effort=500 velocity=1 -> lower=-6.28 upper=6.28 effort=500 velocity=3.14
- joint Joint2: limit lower=-3.14 upper=3.14 effort=500 velocity=1 -> lower=-6.28 upper=6.28 effort=500 velocity=3.14
- joint Joint3: limit lower=-3.14 upper=3.14 effort=500 velocity=1 -> lower=-6.28 upper=6.28 effort=500 velocity=3.14
- joint Joint4: limit lower=-3.14 upper=3.14 effort=500 velocity=1 -> lower=-6.28 upper=6.28 effort=500 velocity=3.14
- joint Joint5: limit lower=-3.14 upper=3.14 effort=500 velocity=1 -> lower=-6.28 upper=6.28 effort=500 velocity=3.14
- joint Joint6: limit lower=-3.14 upper=3.14 effort=500 velocity=1 -> lower=-6.28 upper=6.28 effort=500 velocity=3.14

Commit message: kuka_urdf.urdf is ok, but move_group_interface does not work

File: ws_kuka/src/kuka_urdf/urdf/kuka_urdf.urdf (robot description, URDF)
Before this commit: robot kuka_urdf, 8 links, 7 joints
Joints:
- joint Joint1: limit lower=-6.28 upper=6.28 effort=500 velocity=3.14 -> lower=-3.14 upper=3.14 effort=500 velocity=3.14
- joint Joint2: limit lower=-6.28 upper=6.28 effort=500 velocity=3.14 -> lower=-3.14 upper=3.14 effort=500 velocity=3.14
- joint Joint3: limit lower=-6.28 upper=6.28 effort=500 velocity=3.14 -> lower=-3.14 upper=3.14 effort=500 velocity=3.14
- joint Joint4: limit lower=-6.28 upper=6.28 effort=500 velocity=3.14 -> lower=-3.14 upper=3.14 effort=500 velocity=3.14
- joint Joint5: limit lower=-6.28 upper=6.28 effort=500 velocity=3.14 -> lower=-3.14 upper=3.14 effort=500 velocity=3.14
- joint Joint6: limit lower=-6.28 upper=6.28 effort=500 velocity=3.14 -> lower=-3.14 upper=3.14 effort=500 velocity=3.14

File: ws_kuka_v2/src/kuka_urdf/urdf/kuka_urdf.urdf (robot description, URDF)
Before this commit: robot kuka_urdf, 7 links, 6 joints
Joints:
- joint Joint1: limit lower=-0.27 upper=0.24 effort=500 velocity=1 -> lower=-0.27 upper=0.24 effort=500 velocity=3.14
- joint Joint2: limit lower=-6.28 upper=6.28 effort=500 velocity=2 -> lower=-3.14 upper=3.14 effort=500 velocity=3.14
- joint Joint3: limit lower=-6.28 upper=6.28 effort=500 velocity=2 -> lower=-3.14 upper=3.14 effort=500 velocity=3.14
- joint Joint4: limit lower=-6.28 upper=6.28 effort=500 velocity=2 -> lower=-3.14 upper=3.14 effort=500 velocity=3.14
- joint Joint5: limit lower=-6.28 upper=6.28 effort=500 velocity=2 -> lower=-3.14 upper=3.14 effort=500 velocity=3.14
- joint Joint6: limit lower=-6.28 upper=6.28 effort=500 velocity=2 -> lower=-3.14 upper=3.14 effort=500 velocity=3.14
