Commit message: ws_kuka_v2 does not work, give it up

File: ws_kuka_v2/src/kuka_urdf/urdf/kuka_urdf.urdf (robot description, URDF)
Before this commit: robot kuka_urdf, 8 links, 7 joints
Links:
- removed link Link7
- link Link6: mass 0.442067197041368 -> 0.45606214626239
Joints:
- removed joint Joint7
- joint Joint1: axis 0 0 0 -> 1 0 0; limit lower=-2 upper=2 effort=0 velocity=1 -> lower=-0.27 upper=0.24 effort=500 velocity=1; type continuous -> prismatic

Commit message: modify versions

File: ws_kuka_v2/src/kuka_urdf/urdf/kuka_urdf.urdf (robot description, URDF)
Before this commit: robot kuka_urdf, 7 links, 6 joints
Links:
- added link Link7, mass 0.0139949492210214; collision mesh filename=package://kuka_urdf/meshes/Link7.STL; visual mesh filename=package://kuka_urdf/meshes/Link7.STL
- link Link6: mass 0.45606214626239 -> 0.442067197041369
Joints:
- added joint Joint7: type revolute, parent Link6, child Link7, origin xyz=0.0665 0 0 rpy=0 0 0, axis 1 0 0, limit lower=-3.14 upper=3.14 effort=500 velocity=3.14
